File: IOT_AIR_FILTER_PROJ_REV_B/IOT_AIR_FILTER_PROJ.kicad_pcb (KiCad board)
At the start: 4 copper layers, 65 x 30 mm, 71 parts, among them J10 Conn_01x05_Socket, J2 Conn_01x02_Socket, J3 Conn_02x20_Odd_Even, J5 Conn_01x04_Pin, J6 Conn_01x04_Pin, J7 Conn_01x04_Pin, J8 Conn_01x04_Pin, J9 Conn_01x04_Pin, U1 AMS1117-5.0, U2 TXS0102DCT, U3 PIC16F18156T-I/SO, U4 MC14051BDR2G, U5 INA180A2, U6 INA180A2, U7 INA180A2, U8 INA180A2, U9 MCP23008-xSO, Y1 Crystal_GND24

Commit message: replaced i2c expander with dedicated LED controller
Parts:
- removed R20, R21, R22, R23, R24, R25, R26, R27: 432, Resistor_SMD:R_0402_1005Metric
- removed U9: MCP23008-xSO, Package_SO:SOIC-18W_7.5x11.6mm_P1.27mm
- added R6: 1k, Resistor_SMD:R_1210_3225Metric, B.Cu at (157.8, 108.4)
- added U10: TLC59108xPW, Package_SO:TSSOP-20_4.4x6.5mm_P0.65mm, B.Cu at (157.8, 113.5)
- turned D10 to 180 degrees
- turned D11 to 180 degrees
- turned D12 to 180 degrees
- turned D5 to 180 degrees
- turned D6 to 180 degrees
- turned D7 to 180 degrees
- turned D8 to 180 degrees
- turned D9 to 180 degrees
Connections:
- D10 pad 1: GND -> Net-(D10-K)
- D10 pad 2: Net-(D10-A) -> +5V
- D11 pad 1: GND -> Net-(D11-K)
- D11 pad 2: Net-(D11-A) -> +5V
- D12 pad 1: GND -> Net-(D12-K)
- D12 pad 2: Net-(D12-A) -> +5V
- D5 pad 1: GND -> Net-(D5-K)
- D5 pad 2: Net-(D5-A) -> +5V
- D6 pad 1: GND -> Net-(D6-K)
- D6 pad 2: Net-(D6-A) -> +5V
- D7 pad 1: GND -> Net-(D7-K)
- D7 pad 2: Net-(D7-A) -> +5V
- D8 pad 1: GND -> Net-(D8-K)
- D8 pad 2: Net-(D8-A) -> +5V
- D9 pad 1: GND -> Net-(D9-K)
- D9 pad 2: Net-(D9-A) -> +5V
- U2 pad 6: unconnected-(U2-OE-Pad6) -> +3.3V
Routing:
- net +5V: track 231.0 -> 286.6 mm
- net Net-(D11-K): track 0.00 -> 49.2 mm, vias 0 -> 2
- net Net-(D12-K): track 0.00 -> 48.8 mm, vias 0 -> 2
- net Net-(D10-K): track 0.00 -> 43.9 mm, vias 0 -> 2
- net Net-(D12-A): track 41.9 -> 0.00 mm, vias 2 -> 0
- net Net-(D11-A): track 40.6 -> 0.00 mm, vias 2 -> 0
- net Net-(D9-K): track 0.00 -> 39.1 mm, vias 0 -> 2
- net Net-(D10-A): track 37.0 -> 0.00 mm, vias 2 -> 0
- net GND: track 125.9 -> 89.3 mm, vias 64 -> 59
- net Net-(D8-K): track 0.00 -> 34.4 mm, vias 0 -> 2
- net Net-(D9-A): track 32.3 -> 0.00 mm, vias 2 -> 0
- net Net-(D7-K): track 0.00 -> 30.5 mm, vias 0 -> 2
- net Net-(D8-A): track 28.5 -> 0.00 mm, vias 2 -> 0
- net Net-(D6-K): track 0.00 -> 28.4 mm, vias 0 -> 2
- net Net-(D5-K): track 0.00 -> 25.6 mm, vias 0 -> 2
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